File: squeezem48a.kicad_pcb (KiCad board)
At the start: 2 copper layers, 19 x 15.9 mm, 15 parts, among them CN1 1u, IC1 ATMEGA48A, J1 AVRISP6, P1 Wi07, P10 GND, P11 GND, P2 OC2B, P3 OC0B, P4 OC0A, P5 OC1B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

Commit message: update to rev A
Parts:
- added Q1: 3VGATE-1A-PMOS, SOT23GDS, F.Cu at (59.3, 56.4)
- moved P6 1.10 mm to (62.6, 58.5)
- moved P1 0.64 mm to (60.3, 62.4)
- moved P9 0.58 mm to (54.6, 61.6)
- moved P3 0.50 mm to (55.5, 65.8)
- moved P10 0.48 mm to (53.9, 63.8)
- moved J1 0.36 mm to (69.9, 68.6)
- moved P4 0.26 mm to (57.1, 67.5)
- moved P5 0.23 mm to (59.4, 68.0)
- moved U1 0.21 mm to (68.5, 57.9)
- moved P7 0.21 mm to (63.6, 60.5)
- moved CN1 0.19 mm to (67.2, 59.0)
- moved P2 0.16 mm to (55.3, 59.4)
- moved IC1 0.15 mm to (59.6, 63.0)
- moved P11 0.14 mm to (62.9, 68.5)
Connections:
- IC1 pad 25: N-000006 (its old number) -> (no net)
- IC1 pad 26: N-000005 (its old number) -> (no net)
- IC1 pad 27: N-000004 -> N-0000011
- IC1 pad 28: N-000003 (its old number) -> N-000004
- IC1 pad 32: (no net) -> N-0000012
- P1 pad 3: N-000005 (its old number) -> N-000008
- P1 pad 4: N-000003 (its old number) -> (no net)
- P1 pad 5: N-000006 (its old number) -> N-0000011
- P1 pad 7: +3.3V -> N-000008
Routing:
- net GND: track 53.5 -> 28.0 mm
- net N-000003 (its old number): track 9.78 -> 0.00 mm, vias 1 -> 0
- net N-000008: track 0.00 -> 9.75 mm, vias 0 -> 2
- net +3.3V: track 38.4 -> 48.0 mm
- net N-000005 (its old number): track 9.37 -> 0.00 mm, vias 1 -> 0
- net N-000006 (its old number): track 7.28 -> 0.00 mm, vias 1 -> 0
- net N-0000012: track 0.00 -> 5.55 mm
- net (no net): track 5.20 -> 0.00 mm
- net N-000003: track 19.8 -> 16.7 mm
- net N-000004: track 11.5 -> 8.80 mm
- net N-0000011: track 0.00 -> 2.38 mm, vias 0 -> 1
- net N-0000015: track 4.01 -> 3.00 mm
Other:
- board text added: "squeezem48a rev A"
- board text removed: "squeezem48a rev -"
