File: squeezem48a.sch (KiCad schematic (older format))
At the start: 15 parts, among them CN1 1u, IC1 ATMEGA48A, J1 AVRISP6, P1 Wi07, P10 GND, P11 GND, P2 OC2B, P3 OC0B, P4 OC0A, P5 OC1B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

Commit message: update to rev A
Parts:
- added Q1: 3VGATE-1A-PMOS, SOT23GDS, symbol MOSFET_P
Connections:
- net +3.3V: now also Q1.D; no longer P1.7
- net at IC1.25 ((PCINT10/ADC2)PC2): no longer P1.5
- net at IC1.26 ((PCINT11/ADC3)PC3): no longer P1.3
- net at IC1.27 ((PCINT12/SDA/ADC4)PC4): now also P1.5; no longer P1.6
- net at IC1.28 ((PCINT14/SCL/ADC5)PC5): now also P1.6; no longer P1.4
- net at IC1.32 ((PCINT18/INT0)PD2): now also Q1.G
- new net: P1.3, P1.7, Q1.S
Changed lines of the file:
@@
 LIBS:ws2812b
 LIBS:zener-sot23-3
+LIBS:squeezem48a-cache
 EELAYER 27 0
 EELAYER END
@@
 Sheet 1 1
 Title "squeezem48a"
-Date "26 sep 2014"
-Rev "-"
+Date "23 oct 2014"
+Rev "A"
 Comp ""
 Comment1 ""
@@
 	1    0    0    -1
 $EndComp
-$Comp
-L +3.3V #PWR014
-U 1 1 5425B084
-P 1100 1300
-F 0 "#PWR014" H 1100 1260 30  0001 C CNN
-F 1 "+3.3V" H 1100 1410 30  0000 C CNN
-F 2 "" H 1100 1300 60  0000 C CNN
-F 3 "" H 1100 1300 60  0000 C CNN
-	1    1100 1300
-	1    0    0    -1
-$EndComp
 Wire Wire Line
 	4400 3950 4150 3950
@@
 	2500 1050 2500 1400
 Wire Wire Line
-	1100 1300 1100 1350
-Wire Wire Line
-	1100 1350 1400 1350
-Wire Wire Line
 	2200 1350 3050 1350
 Wire Wire Line
 	3050 1350 3050 1650
 Wire Wire Line
-	3350 1650 3350 1150
-Wire Wire Line
-	3350 1150 2200 1150
-Wire Wire Line
-	2200 1250 3450 1250
-Wire Wire Line
-	3450 1250 3450 1650
-Wire Wire Line
-	3550 1650 3550 750
-Wire Wire Line
-	3550 750  1300 750
-Wire Wire Line
-	1300 750  1300 1150
-Wire Wire Line
-	1300 1150 1400 1150
-Wire Wire Line
-	1400 1250 1350 1250
-Wire Wire Line
-	1350 1250 1350 800
-Wire Wire Line
-	1350 800  3650 800
-Wire Wire Line
-	3650 800  3650 1650
+	2200 1250 3350 1250
 Wire Wire Line
 	2700 1650 2700 1200
@@
 $EndComp
 $Comp
-L +5V #PWR015
+L +5V #PWR014
 U 1 1 5425B8E8
 P 7400 2350
-F 0 "#PWR015" H 7400 2440 20  0001 C CNN
+F 0 "#PWR014" H 7400 2440 20  0001 C CNN
 F 1 "+5V" H 7400 2440 30  0000 C CNN
 F 2 "" H 7400 2350 60  0000 C CNN
@@
 	7400 2350 7300 2350
 $Comp
-L GND #PWR016
+L GND #PWR015
 U 1 1 5425B949
 P 7450 2500
-F 0 "#PWR016" H 7450 2500 30  0001 C CNN
+F 0 "#PWR015" H 7450 2500 30  0001 C CNN
 F 1 "GND" H 7450 2430 30  0001 C CNN
 F 2 "" H 7450 2500 60  0000 C CNN
@@
 	7450 2450 7450 2500
 $Comp
-L +3.3V #PWR017
+L +3.3V #PWR016
 U 1 1 5425BA07
 P 7550 2650
-F 0 "#PWR017" H 7550 2610 30  0001 C CNN
+F 0 "#PWR016" H 7550 2610 30  0001 C CNN
 F 1 "+3.3V" H 7550 2760 30  0000 C CNN
 F 2 "" H 7550 2650 60  0000 C CNN
@@
 $EndComp
 $Comp
-L GND #PWR018
+L GND #PWR017
 U 1 1 5425C0B6
 P 7300 2050
-F 0 "#PWR018" H 7300 2050 30  0001 C CNN
+F 0 "#PWR017" H 7300 2050 30  0001 C CNN
 F 1 "GND" H 7300 1980 30  0001 C CNN
 F 2 "" H 7300 2050 60  0000 C CNN
@@
 Wire Wire Line
 	7150 2050 7300 2050
+$Comp
+L MOSFET_P Q1
+U 1 1 5449305A
+P 1650 2000
+F 0 "Q1" H 1650 2190 60  0000 R CNN
+F 1 "3VGATE-1A-PMOS" H 1650 1820 60  0000 R CNN
+F 2 "SOT23GDS" H 1650 2000 60  0000 C CNN
+F 3 "~" H 1650 2000 60  0000 C CNN
+	1    1650 2000
+	1    0    0    -1
+$EndComp
+$Comp
+L +3.3V #PWR018
+U 1 1 5449310F
+P 1750 1700
+F 0 "#PWR018" H 1750 1660 30  0001 C CNN
+F 1 "+3.3V" H 1750 1810 30  0000 C CNN
+F 2 "" H 1750 1700 60  0000 C CNN
+F 3 "" H 1750 1700 60  0000 C CNN
+	1    1750 1700
+	1    0    0    -1
+$EndComp
+Wire Wire Line
+	1950 2200 1750 2200
+Wire Wire Line
+	1750 1700 1750 1800
+Wire Wire Line
+	1950 2200 1950 1450
+Wire Wire Line
+	1950 1450 1300 1450
+Wire Wire Line
+	1300 1450 1300 1150
+Wire Wire Line
+	1300 1350 1400 1350
+Wire Wire Line
+	950  950  3450 950
+Wire Wire Line
+	950  950  950  1250
+Wire Wire Line
+	950  1250 1400 1250
+Wire Wire Line
+	2100 1600 2100 2450
+Wire Wire Line
+	2100 2450 1450 2450
+Wire Wire Line
+	1450 2450 1450 2000
+Wire Wire Line
+	2950 1650 2950 1600
+Wire Wire Line
+	2950 1600 2100 1600
+Wire Wire Line
+	1300 1150 1400 1150
+Connection ~ 1300 1350
+Wire Wire Line
+	3350 1250 3350 1650
+Wire Wire Line
+	3450 950  3450 1650
 $EndSCHEMATC
